Commit message: Imported upstream version '1.1.2' of 'upstream'

File: urdf/all_sensors.urdf.xacro (robot description, xacro)
@@ -16,4 +16,6 @@
   <!-- Hokuyo ust10lx -->
   <xacro:include filename="$(find robotnik_sensors)/urdf/hokuyo_ust10lx.urdf.xacro" />
+   <!-- Hokuyo ust20lx -->
+  <xacro:include filename="$(find robotnik_sensors)/urdf/hokuyo_ust20lx.urdf.xacro" />
   <!-- Imu -->
   <xacro:include filename="$(find robotnik_sensors)/urdf/imu.urdf.xacro" />
@@ -32,11 +34,23 @@
   <!-- KinectV2 -->
   <xacro:include filename="$(find robotnik_sensors)/urdf/kinectv2.urdf.xacro" />
+  <!-- Sick Tim 551 -->
+  <xacro:include filename="$(find robotnik_sensors)/urdf/sick_tim551.urdf.xacro" />
   <!-- Sick Tim 571 -->
   <xacro:include filename="$(find robotnik_sensors)/urdf/sick_tim571.urdf.xacro" />
+  <!-- Sick Tim 551 -->
+  <xacro:include filename="$(find robotnik_sensors)/urdf/sick_tim551.urdf.xacro" />
   <!-- Orbbec Astra -->
   <xacro:include filename="$(find robotnik_sensors)/urdf/orbbec_astra.urdf.xacro" />
   <!-- Rplidar -->
   <xacro:include filename="$(find robotnik_sensors)/urdf/rplidar.urdf.xacro" />
+  <!-- Rplidar A2 -->
+  <xacro:include filename="$(find robotnik_sensors)/urdf/rplidar_a2.urdf.xacro" />
+  <!-- Rplidar A2 -->
+  <xacro:include filename="$(find robotnik_sensors)/urdf/rplidar_a2.urdf.xacro" />
   <!-- uEye CP Gige -->
   <xacro:include filename="$(find robotnik_sensors)/urdf/ueye_cp_gige.urdf.xacro" />
+  <!-- Pointgrey Bumblebee -->
+  <xacro:include filename="$(find robotnik_sensors)/urdf/pointgrey_bumblebee2.urdf.xacro" />
+  <!-- Intel Realsense D435 -->
+  <xacro:include filename="$(find robotnik_sensors)/urdf/intel_d435.urdf.xacro" />
 </robot>

File: urdf/axis_m5013.urdf.xacro (robot description, xacro)
@@ -6,15 +6,13 @@
   <xacro:property name="ptz_joint_damping" value="0.1"/>
   <xacro:property name="ptz_mechanical_reduction" value="1.0"/>
-  <xacro:macro name="sensor_axis_m5013" params="name parent *origin">
-    <joint name="${name}_joint" type="fixed">
+  <xacro:property name="PI" value="3.14159265359"/>
+  <xacro:macro name="sensor_axis_m5013" params="prefix parent *origin">
+    <joint name="${prefix}_joint" type="fixed">
       <axis xyz="0 1 0"/>
-      <!--
-	      <origin xyz="0.180 0.0 0.270"/>
--->
       <xacro:insert_block name="origin"/>
       <parent link="${parent}"/>
-      <child link="${name}_link"/>
+      <child link="${prefix}_base_link"/>
     </joint>
-    <link name="${name}_link">
+    <link name="${prefix}_base_link">
       <inertial>
         <origin xyz="0 0 0" rpy="0 0 0"/>
@@ -40,14 +38,14 @@
       </collision>
     </link>
-    <joint name="joint_${name}_pan" type="revolute">
-      <axis xyz="0 0 -1"/>
+    <joint name="${prefix}_pan_joint" type="revolute">
+      <axis xyz="1 0 0"/>
       <origin xyz="0.04 0.0 0.0" rpy="0 0 0"/>
       <!-- check the displacement -->
-      <parent link="${name}_link"/>
-      <child link="${name}_pan_link"/>
+      <parent link="${prefix}_base_link"/>
+      <child link="${prefix}_pan_link"/>
       <limit effort="${ptz_joint_effort_limit}" velocity="${ptz_joint_velocity_limit}" lower="-3.1416" upper="3.1416"/>
       <joint_properties damping="${ptz_joint_damping}" friction="{ptz_joint_friction}"/>
     </joint>
-    <link name="${name}_pan_link">
+    <link name="${prefix}_pan_link">
       <inertial>
         <mass value="0.1"/>
@@ -56,23 +54,23 @@
       </inertial>
     </link>
-    <transmission name="${name}_pan_trans">
+    <transmission name="${prefix}_pan_trans">
       <type>transmission_interface/SimpleTransmission</type>
-      <joint name="joint_${name}_pan">
-        <hardwareInterface>PositionJointInterface</hardwareInterface>
+      <joint name="${prefix}_pan_joint">
+        <hardwareInterface>hardware_interface/PositionJointInterface</hardwareInterface>
       </joint>
-      <actuator name="pan_motor">
-        <hardwareInterface>PositionJointInterface</hardwareInterface>
+      <actuator name="${prefix}pan_motor">
+        <hardwareInterface>hardware_interface/PositionJointInterface</hardwareInterface>
         <mechanicalReduction>${ptz_mechanical_reduction}</mechanicalReduction>
       </actuator>
     </transmission>
-    <joint name="joint_${name}_tilt" type="revolute">
+    <joint name="${prefix}_tilt_joint" type="revolute">
       <axis xyz="0 -1 0"/>
-      <origin xyz="0.0 0.0 0.0"/>
-      <parent link="${name}_pan_link"/>
-      <child link="${name}_tilt_link"/>
+      <origin xyz="0.0 0.0 0.0" rpy="0 ${-PI/2} 0"/>
+      <parent link="${prefix}_pan_link"/>
+      <child link="${prefix}_tilt_link"/>
       <limit effort="${ptz_joint_effort_limit}" velocity="${ptz_joint_velocity_limit}" lower="-1.5708" upper="1.5708"/>
       <joint_properties damping="${ptz_joint_damping}" friction="{ptz_joint_friction}"/>
     </joint>
-    <link name="${name}_tilt_link">
+    <link name="${prefix}_tilt_link">
       <inertial>
         <mass value="0.1"/>
@@ -81,20 +79,20 @@
       </inertial>
     </link>
-    <transmission name="${name}_tilt_trans">
+    <transmission name="${prefix}_tilt_trans">
       <type>transmission_interface/SimpleTransmission</type>
-      <joint name="joint_${name}_tilt">
-        <hardwareInterface>PositionJointInterface</hardwareInterface>
+      <joint name="${prefix}_tilt_joint">
+        <hardwareInterface>hardware_interface/PositionJointInterface</hardwareInterface>
       </joint>
-      <actuator name="tilt_motor">
-        <hardwareInterface>PositionJointInterface</hardwareInterface>
+      <actuator name="${prefix}tilt_motor">
+        <hardwareInterface>hardware_interface/PositionJointInterface</hardwareInterface>
         <mechanicalReduction>${ptz_mechanical_reduction}</mechanicalReduction>
       </actuator>
     </transmission>
-    <joint name="${name}_frame_joint" type="fixed">
+    <joint name="${prefix}_frame_joint" type="fixed">
       <origin xyz="0 0 0" rpy="0 0 0"/>
-      <parent link="${name}_tilt_link"/>
-      <child link="${name}_frame"/>
+      <parent link="${prefix}_tilt_link"/>
+      <child link="${prefix}_frame_link"/>
     </joint>
-    <link name="${name}_frame">
+    <link name="${prefix}_frame_link">
       <inertial>
         <mass value="0.001"/>
@@ -104,10 +102,10 @@
     </link>
     <!-- Optical frame -->
-    <joint name="${name}_optical_joint" type="fixed">
+    <joint name="${prefix}_optical_joint" type="fixed">
       <origin xyz="0 0 0" rpy="${-M_PI/2} 0 ${-M_PI/2}"/>
-      <parent link="${name}_frame"/>
-      <child link="${name}_optical_frame"/>
+      <parent link="${prefix}_frame_link"/>
+      <child link="${prefix}_optical_frame_link"/>
     </joint>
-    <link name="${name}_optical_frame">
+    <link name="${prefix}_optical_frame_link">
       <inertial>
         <mass value="0.001"/>
@@ -116,5 +114,5 @@
       </inertial>
     </link>
-    <gazebo reference="${name}_link">
+    <gazebo reference="${prefix}_base_link">
       <material>Gazebo/FlatBlack</material>
     </gazebo>
@@ -123,8 +121,8 @@
   </xacro:macro>
 	<xacro:macro name="sensor_axis_m5013_gazebo">
-		<gazebo reference="${name}_frame"> <!-- the image will be generated from this (${name}_frame) point of view, with the front being the X axis -->
-			<sensor type="camera" name="${name}_sensor">
+		<gazebo reference="${prefix}_frame_link"> <!-- the image will be generated from this (${name}_frame) point of view, with the front being the X axis -->
+			<sensor type="camera" name="${prefix}_sensor">
 				<update_rate>30.0</update_rate>
-				<camera name="${name}">
+				<camera name="${prefix}">
 					<horizontal_fov>${60.0*M_PI/180.0}</horizontal_fov>
 					<image>
@@ -138,12 +136,12 @@
 					</clip>
 				</camera>
-				<plugin name="${name}_controller" filename="libgazebo_ros_camera.so">
-				    <cameraName>${name}</cameraName>
+				<plugin name="${prefix}_controller" filename="libgazebo_ros_camera.so">
+				    <cameraName>${prefix}</cameraName>
 					<alwaysOn>true</alwaysOn>
 					<updateRate>0.0</updateRate>
-					<cameraName>${name}</cameraName>
+					<cameraName>${prefix}</cameraName>
 					<imageTopicName>image_raw</imageTopicName>
 					<cameraInfoTopicName>camera_info</cameraInfoTopicName>
-					<frameName>${name}_optical_frame</frameName>
+					<frameName>${prefix}_optical_frame_link</frameName>
 					<!-- this is just which name the Image msg will have, it does not affect the simulation.
 					     However must be set to the optical_frame,  -->
@@ -154,4 +152,5 @@
 					<distortionT1>0.0</distortionT1>
 					<distortionT2>0.0</distortionT2>
+					<ignoreTfPrefix>1</ignoreTfPrefix>
 				</plugin>
 			</sensor>

File: urdf/hokuyo_ust20lx.urdf.xacro (robot description, xacro)
@@ -1,5 +1,6 @@
 <?xml version="1.0"?>
-<robot xmlns:xacro="http://www.ros.org/wiki/xacro">
-  <xacro:macro name="sensor_sick_tim571" params="prefix parent prefix_topic:='front_laser' *origin min_angle:=-2.36 max_angle:=2.36">
+<robot name="sensor_hokuyo_ust20lx" xmlns:xacro="http://www.ros.org/wiki/xacro">
+  <xacro:macro name="sensor_hokuyo_ust20lx" params="prefix parent prefix_topic:='front_laser' *origin min_angle:=-2.3562 max_angle:=2.3562">
+			<!--arg name="namespace" value="$(arg namespace)"/-->
     <joint name="${prefix}_base_joint" type="fixed">
       <xacro:insert_block name="origin" />
@@ -9,13 +10,13 @@
     <link name="${prefix}_base_link">
       <collision>
-        <origin xyz="0 0 0" rpy="0 0 0"/>
+        <origin xyz="0 0 -0.05" rpy="0 0 0"/>
         <geometry>
-         <mesh filename="package://robotnik_sensors/meshes/sick_tim571.dae"/>
+          <box size="0.010 0.010 0.010"/>
         </geometry>
       </collision>
       <visual>
-        <origin xyz="0 0 0" rpy="0 0 0"/>
+        <origin xyz="0 0 -0.05" rpy="0 0 0"/>
         <geometry>
-            <mesh filename="package://robotnik_sensors/meshes/sick_tim571.dae"/>
+            <mesh filename="package://robotnik_sensors/meshes/hokuyo_ust_20lx.dae"/>
         </geometry>
       </visual>
@@ -26,23 +27,24 @@
       </inertial>
     </link>
+    <link name="${prefix}_link">
+	</link>
     <joint name="${prefix}_joint" type="fixed">
-      <origin xyz="0 0 0.06246" rpy="0 0 0"/>
       <parent link="${prefix}_base_link"/>
       <child link="${prefix}_link"/>
-    </joint>
-    <link name="${prefix}_link">
-    </link>
-    <sensor_sick_tim571_gazebo/>
+      <origin xyz="0.00 0 0.0" rpy="0 0 0"/>
+	</joint>
+    <!-- Hokuyo sensor for simulation -->
+    <xacro:sensor_hokuyo_ust20_gazebo/>
   </xacro:macro>
-  <xacro:macro name="sensor_sick_tim571_gazebo">
-	<gazebo reference="${prefix}_link">
+  <xacro:macro name="sensor_hokuyo_ust20_gazebo">
+    <gazebo reference="${prefix}_link">
 			<sensor type="ray" name="${prefix}_sensor">
 				<pose>0 0 0 0 0 0</pose>
 				<visualize>false</visualize>
-				<update_rate>15</update_rate>
+				<update_rate>40</update_rate>
 				<ray>
 					<scan>
 						<horizontal>
-							<samples>819</samples>
+							<samples>1081</samples>
 							<resolution>1</resolution>
 							<min_angle>${min_angle}</min_angle>
@@ -51,7 +53,9 @@
 					</scan>
 					<range>
-						<min>0.05</min>
-						<max>25.0</max>
-						<resolution>0.00575</resolution>
+						<min>0.06</min>
+						<max>20.0</max>
+						<!-- resolution>0.004363323</resolution -->
+						<resolution>0.004359297</resolution>
+						<!-- resolution>0.001</resolution -->
 					</range>
 					<noise>

File: urdf/rplidar_a2.urdf.xacro (robot description, xacro)
@@ -1,15 +1,15 @@
 <?xml version="1.0"?>
 <robot xmlns:xacro="http://www.ros.org/wiki/xacro">
-  <xacro:macro name="sensor_rplidar" params="prefix parent prefix_topic:='front_laser' *origin min_angle:=3.14159 max_angle:=-3.14159">
-    <joint name="${prefix}_laser_base_joint" type="fixed">
+  <xacro:macro name="sensor_rplidar_a2" params="prefix parent prefix_topic:='front_laser' *origin min_angle:=-3.14159 max_angle:=3.14159">
+    <joint name="${prefix}_base_joint" type="fixed">
       <xacro:insert_block name="origin" />
       <parent link="${parent}"/>
-      <child link="${prefix}_laser_base_link"/>
+      <child link="${prefix}_base_link"/>
     </joint>
-    <link name="${prefix}_laser_base_link">
+    <link name="${prefix}_base_link">
       <collision>
         <origin xyz="0 0 0" rpy="0 0 0"/>
         <geometry>
-         <mesh filename="package://robotnik_sensors/meshes/rplidar.dae"/>
+         <mesh filename="package://robotnik_sensors/meshes/rplidar_a2.dae"/>
         </geometry>
       </collision>
@@ -17,5 +17,5 @@
         <origin xyz="0 0 0" rpy="0 0 0"/>
         <geometry>
-            <mesh filename="package://robotnik_sensors/meshes/rplidar.dae"/>
+            <mesh filename="package://robotnik_sensors/meshes/rplidar_a2.dae"/>
         </geometry>
       </visual>
@@ -27,15 +27,15 @@
     </link>
     <joint name="${prefix}_laser_joint" type="fixed">
-      <origin xyz="0 0 0.0461" rpy="0 0 0"/>
-      <parent link="${prefix}_laser_base_link"/>
-      <child link="${prefix}_laser_link"/>
+      <origin xyz="0 0 0.03086" rpy="0 0 3.1415"/>
+      <parent link="${prefix}_base_link"/>
+      <child link="${prefix}_link"/>
     </joint>
-    <link name="${prefix}_laser_link">
+    <link name="${prefix}_link">
     </link>
-    <sensor_rplidar_gazebo/>
+    <sensor_rplidar_a2_gazebo/>
   </xacro:macro>
-  <xacro:macro name="${prefix}_sensor_rplidar_gazebo">
-    <gazebo reference="${prefix}_laser_link">
-			<sensor type="ray" name="${prefix}_rplidar_sensor">
+  <xacro:macro name="sensor_rplidar_a2_gazebo">
+    <gazebo reference="${prefix}_link">
+			<sensor type="ray" name="${prefix}_rplidar_a2_sensor">
 				<pose>0 0 0 0 0 0</pose>
 				<visualize>false</visualize>
@@ -45,5 +45,5 @@
 						<horizontal>
 							<samples>361</samples>
-							<resolution>1</resolution>
+							<resolution>0.9</resolution>
 							<min_angle>${min_angle}</min_angle>
 							<max_angle>${max_angle}</max_angle>
@@ -61,7 +61,7 @@
 					</noise>
 				</ray>
-				<plugin name="gazebo_ros_rplidar_controller" filename="libgazebo_ros_laser.so">
+				<plugin name="${prefix}gazebo_ros_rplidar_a2_controller" filename="libgazebo_ros_laser.so">
 					<topicName>${prefix_topic}/scan</topicName>
-					<frameName>/${prefix}_laser_link</frameName>
+					<frameName>/${prefix}_link</frameName>
 				</plugin>
 			</sensor>

File: urdf/sick_tim551.urdf.xacro (robot description, xacro)
@@ -1,15 +1,15 @@
 <?xml version="1.0"?>
 <robot xmlns:xacro="http://www.ros.org/wiki/xacro">
-  <xacro:macro name="sensor_rplidar" params="prefix parent prefix_topic:='front_laser' *origin min_angle:=3.14159 max_angle:=-3.14159">
-    <joint name="${prefix}_laser_base_joint" type="fixed">
+  <xacro:macro name="sensor_sick_tim551" params="prefix parent prefix_topic:='front_laser' *origin min_angle:=-2.36 max_angle:=2.36">
+    <joint name="${prefix}_base_joint" type="fixed">
       <xacro:insert_block name="origin" />
       <parent link="${parent}"/>
-      <child link="${prefix}_laser_base_link"/>
+      <child link="${prefix}_base_link"/>
     </joint>
-    <link name="${prefix}_laser_base_link">
+    <link name="${prefix}_base_link">
       <collision>
         <origin xyz="0 0 0" rpy="0 0 0"/>
         <geometry>
-         <mesh filename="package://robotnik_sensors/meshes/rplidar.dae"/>
+         <mesh filename="package://robotnik_sensors/meshes/sick_tim551.dae"/>
         </geometry>
       </collision>
@@ -17,5 +17,5 @@
         <origin xyz="0 0 0" rpy="0 0 0"/>
         <geometry>
-            <mesh filename="package://robotnik_sensors/meshes/rplidar.dae"/>
+            <mesh filename="package://robotnik_sensors/meshes/sick_tim551.dae"/>
         </geometry>
       </visual>
@@ -26,23 +26,23 @@
       </inertial>
     </link>
-    <joint name="${prefix}_laser_joint" type="fixed">
-      <origin xyz="0 0 0.0461" rpy="0 0 0"/>
-      <parent link="${prefix}_laser_base_link"/>
-      <child link="${prefix}_laser_link"/>
+    <joint name="${prefix}_joint" type="fixed">
+      <origin xyz="0 0 0.06246" rpy="0 0 0"/>
+      <parent link="${prefix}_base_link"/>
+      <child link="${prefix}_link"/>
     </joint>
-    <link name="${prefix}_laser_link">
+    <link name="${prefix}_link">
     </link>
-    <sensor_rplidar_gazebo/>
+    <sensor_sick_tim551_gazebo/>
   </xacro:macro>
-  <xacro:macro name="${prefix}_sensor_rplidar_gazebo">
-    <gazebo reference="${prefix}_laser_link">
-			<sensor type="ray" name="${prefix}_rplidar_sensor">
+  <xacro:macro name="sensor_sick_tim551_gazebo">
+    <gazebo reference="${prefix}_link">
+			<sensor type="ray" name="${prefix}_sensor">
 				<pose>0 0 0 0 0 0</pose>
 				<visualize>false</visualize>
-				<update_rate>10</update_rate>
+				<update_rate>15</update_rate>
 				<ray>
 					<scan>
 						<horizontal>
-							<samples>361</samples>
+							<samples>819</samples>
 							<resolution>1</resolution>
 							<min_angle>${min_angle}</min_angle>
@@ -51,7 +51,7 @@
 					</scan>
 					<range>
-						<min>0.15</min>
-						<max>6.0</max>
-						<resolution>0.0174</resolution>
+						<min>0.05</min>
+						<max>10.0</max>
+						<resolution>0.01745</resolution>
 					</range>
 					<noise>
@@ -61,7 +61,7 @@
 					</noise>
 				</ray>
-				<plugin name="gazebo_ros_rplidar_controller" filename="libgazebo_ros_laser.so">
+				<plugin name="${prefix}_controller" filename="libgazebo_ros_laser.so">
 					<topicName>${prefix_topic}/scan</topicName>
-					<frameName>/${prefix}_laser_link</frameName>
+					<frameName>/${prefix}_link</frameName> <!-- leading / avoids that current namespace is added as prefix in the frame name (/ns/prefix_link) -->
 				</plugin>
 			</sensor>
