Commit message: Imported upstream version '1.12.0' of 'upstream'

File: urdf/all_sensors.urdf.xacro (robot description, xacro)
@@ -1,9 +1,12 @@
 <?xml version="1.0"?>
-<robot name="all_sensors" xmlns:xacro="http://www.ros.org/wiki/xacro">
-	<!-- This file unifies all sensors that can be used on simulation, defined as xacro:macros -->
+<robot name="all_sensors"
+  xmlns:xacro="http://wiki.ros.org/xacro">
+  <!-- This file unifies all sensors that can be used on simulation, defined as xacro:macros -->
   <!-- Axis p5512 -->
   <xacro:include filename="$(find robotnik_sensors)/urdf/axis.urdf.xacro" />
   <!-- Axis m5013 -->
   <xacro:include filename="$(find robotnik_sensors)/urdf/axis_m5013.urdf.xacro" />
+  <!-- Axis m5525 -->
+  <xacro:include filename="$(find robotnik_sensors)/urdf/axis_m5525.urdf.xacro" />
   <!-- Fotonic E Series -->
   <xacro:include filename="$(find robotnik_sensors)/urdf/fotonic_e.urdf.xacro" />
@@ -16,5 +19,7 @@
   <!-- Hokuyo ust10lx -->
   <xacro:include filename="$(find robotnik_sensors)/urdf/hokuyo_ust10lx.urdf.xacro" />
-   <!-- Hokuyo ust20lx -->
+  <!-- Hokuyo ust20lx -->
+  <xacro:include filename="$(find robotnik_sensors)/urdf/hokuyo_ust20lx.urdf.xacro" />
+  <!-- Hokuyo ust20lx -->
   <xacro:include filename="$(find robotnik_sensors)/urdf/hokuyo_ust20lx.urdf.xacro" />
   <!-- Imu -->
@@ -32,4 +37,6 @@
   <!-- Sick s300 -->
   <xacro:include filename="$(find robotnik_sensors)/urdf/sick_s300.urdf.xacro" />
+  <!-- Sick microscan3 -->
+  <xacro:include filename="$(find robotnik_sensors)/urdf/sick_microscan3.urdf.xacro" />
   <!-- KinectV2 -->
   <xacro:include filename="$(find robotnik_sensors)/urdf/kinectv2.urdf.xacro" />
@@ -42,4 +49,6 @@
   <!-- Orbbec Astra -->
   <xacro:include filename="$(find robotnik_sensors)/urdf/orbbec_astra.urdf.xacro" />
+  <!-- Zed -->
+  <xacro:include filename="$(find robotnik_sensors)/urdf/zed.urdf.xacro" />
   <!-- Rplidar -->
   <xacro:include filename="$(find robotnik_sensors)/urdf/rplidar.urdf.xacro" />
@@ -52,5 +61,19 @@
   <!-- Pointgrey Bumblebee -->
   <xacro:include filename="$(find robotnik_sensors)/urdf/pointgrey_bumblebee2.urdf.xacro" />
+  <!-- Intel Realsense R430 -->
+  <xacro:include filename="$(find robotnik_sensors)/urdf/intel_r430.urdf.xacro" />
   <!-- Intel Realsense D435 -->
   <xacro:include filename="$(find robotnik_sensors)/urdf/intel_d435.urdf.xacro" />
+  <!-- Velodyne VLP16 -->
+  <xacro:include filename="$(find robotnik_sensors)/urdf/velodyne_vlp16.urdf.xacro" />
+  <!-- Teraranger Duo-->
+  <xacro:include filename="$(find robotnik_sensors)/urdf/teraranger_tr_duo.urdf.xacro" />
+  <!-- Roboteq MGS -->
+  <xacro:include filename="$(find robotnik_sensors)/urdf/roboteq_mgs.urdf.xacro" />
+  <!-- Benewake CE-30 (all, includes a, c and d) -->
+  <xacro:include filename="$(find robotnik_sensors)/urdf/benewake_ce30.urdf.xacro" />
+  <!-- Rubedos Viper -->
+  <xacro:include filename="$(find robotnik_sensors)/urdf/rubedos_viper.urdf.xacro" />
+  <!-- RoboSense RS-Lidar -->
+  <xacro:include filename="$(find robotnik_sensors)/urdf/rslidar.urdf.xacro" />
 </robot>

File: urdf/axis.urdf.xacro (robot description, xacro)
@@ -1,4 +1,4 @@
 <?xml version="1.0"?>
-<robot xmlns:xacro="http://www.ros.org/wiki/xacro" name="sensor_axis">
+<robot xmlns:xacro="http://wiki.ros.org/xacro" name="sensor_axis">
   <xacro:property name="ptz_joint_effort_limit" value="100.0"/>
   <xacro:property name="ptz_joint_velocity_limit" value="100.0"/>
@@ -6,5 +6,5 @@
   <xacro:property name="ptz_joint_damping" value="0.1"/>
   <xacro:property name="ptz_mechanical_reduction" value="1.0"/>
-  <xacro:macro name="sensor_axis" params="prefix parent *origin">
+  <xacro:macro name="sensor_axis" params="prefix parent *origin far:=^|8.0 near:=^|0.05">
     <joint name="${prefix}_joint" type="fixed">
       <axis xyz="0 1 0"/>
@@ -44,5 +44,5 @@
       <parent link="${prefix}_base_link"/>
       <child link="${prefix}_pan_link"/>
-      <limit effort="${ptz_joint_effort_limit}" velocity="${ptz_joint_velocity_limit}" lower="-3.1416" upper="3.1416"/>
+      <limit effort="${ptz_joint_effort_limit}" velocity="${ptz_joint_velocity_limit}" lower="-3.1415" upper="3.1415"/>
       <joint_properties damping="${ptz_joint_damping}" friction="{ptz_joint_friction}"/>
     </joint>
@@ -57,8 +57,8 @@
       <type>transmission_interface/SimpleTransmission</type>
       <joint name="${prefix}_pan_joint">
-        <hardwareInterface>hardware_interface/PositionJointInterface</hardwareInterface>
+        <hardwareInterface>hardware_interface/VelocityJointInterface</hardwareInterface>
       </joint>
       <actuator name="pan_motor">
-        <hardwareInterface>hardware_interface/PositionJointInterface</hardwareInterface>
+        <hardwareInterface>hardware_interface/VelocityJointInterface</hardwareInterface>
         <mechanicalReduction>${ptz_mechanical_reduction}</mechanicalReduction>
       </actuator>
@@ -82,8 +82,8 @@
       <type>transmission_interface/SimpleTransmission</type>
       <joint name="${prefix}_tilt_joint">
-        <hardwareInterface>hardware_interface/PositionJointInterface</hardwareInterface>
+        <hardwareInterface>hardware_interface/VelocityJointInterface</hardwareInterface>
       </joint>
       <actuator name="tilt_motor">
-        <hardwareInterface>hardware_interface/PositionJointInterface</hardwareInterface>
+        <hardwareInterface>hardware_interface/VelocityJointInterface</hardwareInterface>
         <mechanicalReduction>${ptz_mechanical_reduction}</mechanicalReduction>
       </actuator>
@@ -132,6 +132,6 @@
           </image>
           <clip>
-            <near>0.05</near>
-            <far>8.0</far>
+            <near>${near}</near>
+            <far>${far}</far>
           </clip>
         </camera>

File: urdf/gps.urdf.xacro (robot description, xacro)
@@ -1,5 +1,6 @@
 <?xml version="1.0"?>
-<robot name="sensor_gps" xmlns:xacro="http://www.ros.org/wiki/xacro">
-  <xacro:macro name="sensor_gps" params="prefix parent *origin">
+<robot name="sensor_gps" xmlns:xacro="http://wiki.ros.org/xacro">
+  <!-- if no latitude/longitud is specified, then use Fuente del Jarro as default -->
+  <xacro:macro name="sensor_gps" params="prefix parent *origin gps_latitude:=^|39.5080331 gps_longitude:=^|-0.4619816 update_rate:=^|5">
 	  <!-- ANTENNA GPS -->
 	  <joint name="${prefix}_joint" type="fixed">
@@ -38,18 +39,18 @@
       <plugin name="${prefix}_controller" filename="libhector_gazebo_ros_gps.so">
         <alwaysOn>1</alwaysOn>
-        <updateRate>5</updateRate>
+        <updateRate>${update_rate}</updateRate>
         <bodyName>${prefix}_base_link</bodyName> <!-- must be the link of the gps device, not the base_link or base_footprint -->
-        <frameId>/${prefix}_base_link</frameId>
-        <topicName>fix</topicName>
-        <!-- Robotnik position at Fuente del Jarro -->
-        <referenceLatitude>39.5080331</referenceLatitude>
-        <referenceLongitude>-0.4619816</referenceLongitude>
+        <frameId>${prefix}_base_link</frameId>
+        <topicName>gps/fix</topicName>
+        <!-- GPS coordinates -->
+        <referenceLatitude>${gps_latitude}</referenceLatitude>
+        <referenceLongitude>${gps_longitude}</referenceLongitude>
         <!-- To set heading in ENU orientation (degrees) -->
         <referenceHeading>90</referenceHeading>
-        <velocityTopicName>fix_velocity</velocityTopicName>
+        <velocityTopicName>gps/fix_velocity</velocityTopicName>
         <drift>0.0 0.0 0.0</drift>
         <!--<drift>0.0001 0.0001 0.0001</drift>-->
         <!--<drift>0.3 0.3 0.3</drift>-->
-        <gaussianNoise>0.1 0.1 0.1</gaussianNoise>
+        <gaussianNoise>0.00001 0.00001 0.00001</gaussianNoise>
         <!--<gaussianNoise>0.00001 0.00001 0.00001</gaussianNoise>-->
         <velocityDrift>0.00001 0.00001 0.00001</velocityDrift>

File: urdf/hokuyo_utm30lx.urdf.xacro (robot description, xacro)
@@ -1,5 +1,5 @@
 <?xml version="1.0"?>
-<robot name="sensor_hokuyo_utm30lx" xmlns:xacro="http://www.ros.org/wiki/xacro">
-  <xacro:macro name="sensor_hokuyo_utm30lx" params="prefix parent prefix_topic:='front_laser *origin min_angle:=-2.35 max_angle:=2.35">
+<robot name="sensor_hokuyo_utm30lx" xmlns:xacro="http://wiki.ros.org/xacro">
+  <xacro:macro name="sensor_hokuyo_utm30lx" params="prefix parent prefix_topic:='front_laser' *origin min_angle:=-2.35 max_angle:=2.35 gpu:=^|true">
     <joint name="${prefix}_base_joint" type="fixed">
       <!-- FRONT MOUNT  -->
@@ -36,5 +36,13 @@
   <xacro:macro name="sensor_hokuyo_utm_gazebo">
     <gazebo reference="${prefix}_link">
-			<sensor type="ray" name="${prefix}_sensor">
+			<xacro:if value="${gpu}">
+        <xacro:property name="ray_type" value="gpu_ray" />
+        <xacro:property name="plugin_lib" value="libgazebo_ros_gpu_laser.so" />
+      </xacro:if>
+      <xacro:unless value="${gpu}">
+        <xacro:property name="ray_type" value="ray" />
+        <xacro:property name="plugin_lib" value="libgazebo_ros_laser.so" />
+      </xacro:unless>
+			<sensor type="${ray_type}" name="${prefix}_sensor">
 				<pose>0 0 0 0 0 0</pose>
 				<visualize>false</visualize>
@@ -60,5 +68,5 @@
 					</noise>
 				</ray>
-				<plugin name="${prefix}_controller" filename="libgazebo_ros_laser.so">
+				<plugin name="${prefix}_controller" filename="${plugin_lib}">
 					<topicName>${prefix_topic}/scan</topicName>
 					<frameName>/${prefix}_link</frameName>

File: urdf/imu.urdf.xacro (robot description, xacro)
@@ -1,5 +1,5 @@
 <?xml version="1.0"?>
-<robot name="sensor_imu" xmlns:xacro="http://www.ros.org/wiki/xacro">
-  <xacro:macro name="sensor_imu" params="prefix parent *origin">
+<robot name="sensor_imu" xmlns:xacro="http://wiki.ros.org/xacro">
+  <xacro:macro name="sensor_imu" params="prefix ns:='' parent *origin">
 	  <joint name="${prefix}_joint" type="fixed">
 	      <axis xyz="1 0 0"/>
@@ -13,5 +13,5 @@
 	        <mass value="0.001"/>
 	        <origin rpy="0 0 0" xyz="0 0 0"/>
-	        <inertia ixx="0.0001" ixy="0" ixz="0" iyy="0.000001" iyz="0" izz="0.0001"/>
+	        <inertia ixx="0.00000000167" ixy="0" ixz="0" iyy="0.00000000167" iyz="0" izz="0.00000000167"/>
 	      </inertial>
 	      <visual>
@@ -21,20 +21,39 @@
 	        </geometry>
 	      </visual>
-	      <collision>
+	      <!--collision>
 	        <origin rpy="0 0 0" xyz="0 0 0"/>
 	        <geometry>
-	          <box size=".001 .001 .001"/>
+	          <box size="0.001 0.001 0.001"/>
 	        </geometry>
-	      </collision>
+	      </collision-->
 	  </link>
-	  <gazebo>
-	    <plugin name="${prefix}_controller" filename="libgazebo_ros_imu.so">
-	       <topicName>imu/data</topicName>
-	       <serviceName>imu/service</serviceName>
-		   <bodyName>${prefix}_link</bodyName>
-		   <updateRateHZ>50.0</updateRateHZ>
-	       <gaussianNoise>0.005</gaussianNoise>
-	    </plugin>
-	  </gazebo>
+	  <!--<gazebo>-->
+		<!--<plugin name="${prefix}_controller" filename="libgazebo_ros_imu.so">-->
+		   <!--<topicName>${ns}imu/data</topicName>-->
+		   <!--<serviceName>imu/service</serviceName>-->
+		   <!--<bodyName>${prefix}_link</bodyName>-->
+		   <!--<updateRateHZ>50.0</updateRateHZ>-->
+		   <!--<gaussianNoise>0.0</gaussianNoise>-->
+		<!--</plugin>-->
+	  <!--</gazebo>-->
+ <gazebo reference="${prefix}_link">
+    <gravity>true</gravity>
+    <sensor name="${prefix}_imu_sensor" type="imu">
+      <always_on>true</always_on>
+      <update_rate>100</update_rate>
+      <visualize>true</visualize>
+      <topic>__default_topic__</topic>
+      <plugin filename="libgazebo_ros_imu_sensor.so" name="${prefix}_imu_plugin">
+        <topicName>imu/data</topicName>
+		<bodyName>${prefix}_link</bodyName>
+        <updateRateHZ>100.0</updateRateHZ>
+        <gaussianNoise>0.0</gaussianNoise>
+        <xyzOffset>0 0 0</xyzOffset>
+        <rpyOffset>0 0 0</rpyOffset>
+		<frameName>${prefix}_link</frameName>
+      </plugin>
+      <pose>0 0 0 0 0 0</pose>
+    </sensor>
+  </gazebo>
   </xacro:macro>
 </robot>
