Commit message: Imported upstream version '1.12.0' of 'upstream'

File: urdf/sick_s300.urdf.xacro (robot description, xacro)
@@ -1,9 +1,10 @@
 <?xml version="1.0"?>
-<robot name="sensor_sick_s300" xmlns:xacro="http://www.ros.org/wiki/xacro">
-  <xacro:macro name="sensor_sick_s300" params="prefix parent prefix_topic:='front_laser' *origin">
-    <joint name="${prefix}_base_joint" type="fixed">
+<robot name="sensor_sick_s300" xmlns:xacro="http://wiki.ros.org/xacro">
+  <xacro:macro name="sensor_sick_s300" params="prefix parent prefix_topic:='front_laser' *origin min_angle:=-2.3562 max_angle:=2.3562 gpu:=^|true">
+    <joint name="${prefix}_base_joint" type="revolute">
       <xacro:insert_block name="origin" />
       <parent link="${parent}"/>
       <child link="${prefix}_base_link"/>
+      <limit effort="100" velocity="100" lower="0.0" upper="0.0"/>
 	</joint>
 	<link name="${prefix}_base_link">
@@ -22,8 +23,13 @@
 			</geometry>
 		</visual>
-		<inertial>
+		<!--inertial>
 			<mass value="1e-5" />
 			<origin xyz="0 0 0" rpy="0 0 0"/>
 			<inertia ixx="1e-6" ixy="0" ixz="0" iyy="1e-6" iyz="0" izz="1e-6" />
+		</inertial-->
+		<inertial>
+			<mass value="0.1" />
+			<origin xyz="0 0 0" rpy="0 0 0"/>
+			<inertia ixx="0.0002708333" ixy="0" ixz="0" iyy="0.0002708333" iyz="0" izz="0.00009434" />
 		</inertial>
 	</link>
@@ -34,4 +40,14 @@
 	</joint>
 	<link name="${prefix}_link" />
+	<transmission name="${prefix}_base_trans">
+      <type>transmission_interface/SimpleTransmission</type>
+      <joint name="${prefix}_base_joint">
+        <hardwareInterface>hardware_interface/VelocityJointInterface</hardwareInterface>
+      </joint>
+      <actuator name="sick_motor">
+        <hardwareInterface>hardware_interface/VelocityJointInterface</hardwareInterface>
+        <mechanicalReduction>${ptz_mechanical_reduction}</mechanicalReduction>
+      </actuator>
+    </transmission>
 	<!-- Sick sensor sensor for simulation -->
 	<sensor_sick_s300_gazebo />
@@ -39,34 +55,42 @@
   <xacro:macro name="sensor_sick_s300_gazebo">
     <gazebo reference="${prefix}_link">
-			<sensor type="ray" name="${prefix}_sensor">
-				<pose>0 0 0 0 0 0</pose>
-				<visualize>false</visualize>
-				<update_rate>12.5</update_rate>
-				<ray>
-					<scan>
-						<horizontal>
-							<samples>541</samples>
-							<resolution>1</resolution>
-							<min_angle>-2.3562</min_angle>
-							<max_angle>2.3562</max_angle>
-						</horizontal>
-					</scan>
-					<range>
-						<min>0.10</min>
-						<max>30.0</max>
-						<resolution>0.03</resolution>
-					</range>
-					<noise>
-						<type>gaussian</type>
-						<mean>0.0</mean>
-						<stddev>0.03</stddev>
-					</noise>
-				</ray>
-				<plugin name="${prefix}_controller" filename="libgazebo_ros_laser.so">
-					<topicName>${prefix_topic}/scan</topicName>
-					<frameName>/${prefix}_link</frameName><!-- if not global (leading /) sets the current namespace as a prefix (/ns/name_laser_link) -->
-				</plugin>
-			</sensor>
-		</gazebo>
+		<xacro:if value="${gpu}">
+			<xacro:property name="ray_type" value="gpu_ray" />
+			<xacro:property name="plugin_lib" value="libgazebo_ros_gpu_laser.so" />
+		</xacro:if>
+		<xacro:unless value="${gpu}">
+			<xacro:property name="ray_type" value="ray" />
+			<xacro:property name="plugin_lib" value="libgazebo_ros_laser.so" />
+		</xacro:unless>
+		<sensor type="${ray_type}" name="${prefix}_sensor">
+			<pose>0 0 0 0 0 0</pose>
+			<visualize>false</visualize>
+			<update_rate>12.5</update_rate>
+			<ray>
+				<scan>
+					<horizontal>
+						<samples>541</samples>
+						<resolution>1</resolution>
+						<min_angle>${min_angle}</min_angle>
+						<max_angle>${max_angle}</max_angle>
+					</horizontal>
+				</scan>
+				<range>
+					<min>0.10</min>
+					<max>30.0</max>
+					<resolution>0.03</resolution>
+				</range>
+				<noise>
+					<type>gaussian</type>
+					<mean>0.0</mean>
+					<stddev>0.03</stddev>
+				</noise>
+			</ray>
+			<plugin name="${prefix}_controller" filename="${plugin_lib}">
+				<topicName>${prefix_topic}/scan</topicName>
+				<frameName>/${prefix}_link</frameName><!-- if not global (leading /) sets the current namespace as a prefix (/ns/name_laser_link) -->
+			</plugin>
+		</sensor>
+	</gazebo>
   </xacro:macro>
 </robot>
